File: KicadFiles/PlayDice.kicad_pcb (KiCad board)
At the start: 2 copper layers, 40 x 110 mm, 31 parts, among them J1 Clock In, J2 Eurorack_10_pin_power, J3 Action In, J4 OLED, J5 Gate Out, J6 CV Out, Q1 2N3904, Q2 2N3904, SW1 Action Button, SW2 Lane Button, SW3 Right Button, SW4 Left Button, SW5 Rotary_Encoder_Switch, U1 LM1117-5.0, U2 Teensy3.2, U3 TL072

Commit message: Bug fixes and PCB updates
Parts:
- J1, J3, J5, J6: footprint PlayDice:THONKICONN -> PlayDice:THONKICONN_hole
- moved R4 33.9 mm to (138.0, 121.5), turned to 0 degrees
- moved R3 31.6 mm to (138.0, 124.0), turned to 0 degrees
- moved J3 26.0 mm to (136.0, 131.5)
- moved J1 26.0 mm to (136.0, 150.0)
- moved Left1 26.0 mm to (132.0, 89.0)
- moved Right1 26.0 mm to (106.0, 89.0)
- moved Action1 24.5 mm to (107.5, 136.5)
- moved C4 21.6 mm to (124.5, 116.0)
- moved C1 21.5 mm to (116.0, 119.5)
- moved R7 21.0 mm to (121.5, 116.0)
- moved R6 20.0 mm to (106.5, 113.5), turned to 90 degrees
- moved Q2 20.0 mm to (132.5, 121.5), turned to 90 degrees
- moved U1 19.2 mm to (131.0, 114.0)
- moved U3 18.8 mm to (116.0, 113.5)
- moved R2 18.8 mm to (123.0, 142.5), turned to 0 degrees
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- renumbered SW1 to Action1, SW5 to Encoder1, SW2 to Lane1, SW4 to Left1, SW3 to Right1, U2 to Teensy1, Speed1 to Tempo1
Connections:
- Teensy1 pad 10: Net-(U2-Pad10) -> /OLED_DC
- Teensy1 pad 11: Net-(U2-Pad11) -> /OLED_CS
- Teensy1 pad 14: /LEFT -> /RIGHT
- Teensy1 pad 27: /RIGHT -> /ACTION
- Teensy1 pad 29: /ACTION -> /LEFT
- Teensy1 pad 4: /OLED_CS -> Net-(Teensy1-Pad4)
- Teensy1 pad 5: /OLED_DC -> Net-(Teensy1-Pad5)
- Teensy1 pad 6: /OLED_RES -> Net-(Teensy1-Pad6)
- Teensy1 pad 7: /OLED_D1 -> /OLED_D0
- Teensy1 pad 8: /OLED_D0 -> /OLED_D1
- Teensy1 pad 9: Net-(U2-Pad9) -> /OLED_RES
Routing:
- net Net-(J5-Pad3): track 101.0 -> 34.5 mm
- net VCC: track 95.9 -> 46.3 mm
- net Net-(J6-Pad3): track 62.6 -> 37.0 mm
- net GND: track 0.00 -> 25.3 mm, vias 0 -> 1
- net /GATE: track 24.6 -> 48.3 mm
- net +5V: track 33.2 -> 55.5 mm, vias 0 -> 1
- net /CV: track 26.7 -> 47.5 mm, vias 1 -> 0
- net /LEFT: track 22.6 -> 5.88 mm
- net VEE: track 71.3 -> 55.6 mm, vias 2 -> 1
- net +3V3: track 76.1 -> 60.4 mm
- net /RIGHT: track 10.1 -> 22.6 mm
- net /ENC_3: track 31.7 -> 21.6 mm
- net /ENC_SW: track 45.7 -> 37.8 mm
- net /ACTION: track 54.5 -> 62.1 mm
- net /ENC_1: track 30.2 -> 22.7 mm
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Other:
- board text added: "+12"
- board text added: "-12"
