File: KicadFiles/PlayDice.sch (KiCad schematic (older format))
At the start: 31 parts, among them J1 Clock In, J2 Eurorack_10_pin_power, J3 Action In, J4 OLED, J5 Gate Out, J6 CV Out, Q1 2N3904, Q2 2N3904, SW1 Action Button, SW2 Lane Button, SW3 Right Button, SW4 Left Button, SW5 Rotary_Encoder_Switch, U1 LM1117-5.0, U2 Teensy3.2, U3 TL072

Commit message: Bug fixes and PCB updates
Parts:
- renumbered SW1 to Action1, SW5 to Encoder1, SW2 to Lane1, SW4 to Left1, SW3 to Right1, U2 to Teensy1, Speed1 to Tempo1

Commit message: PCB fixed transistor connections; added basic handling for scale quantisation
Parts:
- removed Q1, Q2: 2N3904, TO_SOT_Packages_THT:TO-92_Molded_Narrow, symbol 2N3904
- added Q1, Q2: MMBT3904, TO_SOT_Packages_SMD:SOT-23, symbol MMBT3904
Changed lines of the file:
@@
 $EndComp
 $Comp
-L GND #PWR30
+L GND #PWR01
 U 1 1 5A99E6E6
 P 9900 3950
-F 0 "#PWR30" H 9900 3700 50  0001 C CNN
+F 0 "#PWR01" H 9900 3700 50  0001 C CNN
 F 1 "GND" H 9900 3800 50  0000 C CNN
 F 2 "" H 9900 3950 50  0001 C CNN
@@
 $EndComp
 $Comp
-L +5V #PWR9
+L +5V #PWR02
 U 1 1 5A99E716
 P 4350 2850
-F 0 "#PWR9" H 4350 2700 50  0001 C CNN
+F 0 "#PWR02" H 4350 2700 50  0001 C CNN
 F 1 "+5V" H 4350 2990 50  0000 C CNN
 F 2 "" H 4350 2850 50  0001 C CNN
@@
 $EndComp
 $Comp
-L GND #PWR14
+L GND #PWR03
 U 1 1 5A99E75A
 P 6750 5150
-F 0 "#PWR14" H 6750 4900 50  0001 C CNN
+F 0 "#PWR03" H 6750 4900 50  0001 C CNN
 F 1 "GND" H 6750 5000 50  0000 C CNN
 F 2 "" H 6750 5150 50  0001 C CNN
@@
 $EndComp
 $Comp
-L +3.3V #PWR29
+L +3.3V #PWR04
 U 1 1 5A9AB0CA
 P 9900 3650
-F 0 "#PWR29" H 9900 3500 50  0001 C CNN
+F 0 "#PWR04" H 9900 3500 50  0001 C CNN
 F 1 "+3.3V" H 9900 3790 50  0000 C CNN
 F 2 "" H 9900 3650 50  0001 C CNN
@@
 $EndComp
 $Comp
-L +3.3V #PWR8
+L +3.3V #PWR05
 U 1 1 5A9AB341
 P 4350 2650
-F 0 "#PWR8" H 4350 2500 50  0001 C CNN
+F 0 "#PWR05" H 4350 2500 50  0001 C CNN
 F 1 "+3.3V" H 4350 2790 50  0000 C CNN
 F 2 "" H 4350 2650 50  0001 C CNN
@@
 $EndComp
 $Comp
-L GND #PWR16
+L GND #PWR06
 U 1 1 5A9AB3C0
 P 7850 3650
-F 0 "#PWR16" H 7850 3400 50  0001 C CNN
+F 0 "#PWR06" H 7850 3400 50  0001 C CNN
 F 1 "GND" H 7850 3500 50  0000 C CNN
 F 2 "" H 7850 3650 50  0001 C CNN
@@
 $EndComp
 $Comp
-L GND #PWR11
+L GND #PWR07
 U 1 1 5B3F8B41
 P 6600 1750
-F 0 "#PWR11" H 6600 1500 50  0001 C CNN
+F 0 "#PWR07" H 6600 1500 50  0001 C CNN
 F 1 "GND" H 6600 1600 50  0000 C CNN
 F 2 "" H 6600 1750 50  0001 C CNN
@@
 $EndComp
 $Comp
-L +3.3V #PWR12
+L +3.3V #PWR08
 U 1 1 5B3F8D73
 P 6700 2050
-F 0 "#PWR12" H 6700 1900 50  0001 C CNN
+F 0 "#PWR08" H 6700 1900 50  0001 C CNN
 F 1 "+3.3V" H 6700 2190 50  0000 C CNN
 F 2 "" H 6700 2050 50  0001 C CNN
@@
 $EndComp
 $Comp
-L VCC #PWR6
+L VCC #PWR09
 U 1 1 5B3FD712
 P 3850 2250
-F 0 "#PWR6" H 3850 2100 50  0001 C CNN
+F 0 "#PWR09" H 3850 2100 50  0001 C CNN
 F 1 "VCC" H 3850 2400 50  0000 C CNN
 F 2 "" H 3850 2250 50  0001 C CNN
@@
 $EndComp
 $Comp
-L VEE #PWR7
+L VEE #PWR010
 U 1 1 5B3FD9D0
 P 3850 3500
-F 0 "#PWR7" H 3850 3350 50  0001 C CNN
+F 0 "#PWR010" H 3850 3350 50  0001 C CNN
 F 1 "VEE" H 3850 3650 50  0000 C CNN
 F 2 "" H 3850 3500 50  0001 C CNN
@@
 $EndComp
 $Comp
-L GND #PWR1
+L GND #PWR011
 U 1 1 5B3FDD0F
 P 2650 2850
-F 0 "#PWR1" H 2650 2600 50  0001 C CNN
+F 0 "#PWR011" H 2650 2600 50  0001 C CNN
 F 1 "GND" H 2650 2700 50  0000 C CNN
 F 2 "" H 2650 2850 50  0001 C CNN
@@
 $EndComp
 $Comp
-L VCC #PWR2
+L VCC #PWR012
 U 1 1 5B3FDE28
 P 2900 4200
-F 0 "#PWR2" H 2900 4050 50  0001 C CNN
+F 0 "#PWR012" H 2900 4050 50  0001 C CNN
 F 1 "VCC" H 2900 4350 50  0000 C CNN
 F 2 "" H 2900 4200 50  0001 C CNN
@@
 $EndComp
 $Comp
-L +5V #PWR5
+L +5V #PWR013
 U 1 1 5B3FE23A
 P 3750 4200
-F 0 "#PWR5" H 3750 4050 50  0001 C CNN
+F 0 "#PWR013" H 3750 4050 50  0001 C CNN
 F 1 "+5V" H 3750 4340 50  0000 C CNN
 F 2 "" H 3750 4200 50  0001 C CNN
@@
 $EndComp
 $Comp
-L GND #PWR3
+L GND #PWR014
 U 1 1 5B3FE4FC
 P 3350 4650
-F 0 "#PWR3" H 3350 4400 50  0001 C CNN
+F 0 "#PWR014" H 3350 4400 50  0001 C CNN
 F 1 "GND" H 3350 4500 50  0000 C CNN
 F 2 "" H 3350 4650 50  0001 C CNN
@@
 $EndComp
 $Comp
-L GND #PWR24
+L GND #PWR015
 U 1 1 5B423678
 P 8600 5050
-F 0 "#PWR24" H 8600 4800 50  0001 C CNN
+F 0 "#PWR015" H 8600 4800 50  0001 C CNN
 F 1 "GND" H 8600 4900 50  0000 C CNN
 F 2 "" H 8600 5050 50  0001 C CNN
@@
 $EndComp
 $Comp
-L GND #PWR27
+L GND #PWR016
 U 1 1 5B423A78
 P 9150 5050
-F 0 "#PWR27" H 9150 4800 50  0001 C CNN
+F 0 "#PWR016" H 9150 4800 50  0001 C CNN
 F 1 "GND" H 9150 4900 50  0000 C CNN
 F 2 "" H 9150 5050 50  0001 C CNN
@@
 $EndComp
 $Comp
-L GND #PWR28
+L GND #PWR017
 U 1 1 5B423C16
 P 9250 4100
-F 0 "#PWR28" H 9250 3850 50  0001 C CNN
+F 0 "#PWR017" H 9250 3850 50  0001 C CNN
 F 1 "GND" H 9250 3950 50  0000 C CNN
 F 2 "" H 9250 4100 50  0001 C CNN
@@
 $EndComp
 $Comp
-L GND #PWR15
+L GND #PWR018
 U 1 1 5B425ECA
 P 7850 2250
-F 0 "#PWR15" H 7850 2000 50  0001 C CNN
+F 0 "#PWR018" H 7850 2000 50  0001 C CNN
 F 1 "GND" H 7850 2100 50  0000 C CNN
 F 2 "" H 7850 2250 50  0001 C CNN
@@
 $EndComp
 $Comp
-L GND #PWR25
+L GND #PWR019
 U 1 1 5B42676A
 P 9100 1550
-F 0 "#PWR25" H 9100 1300 50  0001 C CNN
+F 0 "#PWR019" H 9100 1300 50  0001 C CNN
 F 1 "GND" H 9100 1400 50  0000 C CNN
 F 2 "" H 9100 1550 50  0001 C CNN
@@
 $EndComp
 $Comp
-L GND #PWR26
+L GND #PWR020
 U 1 1 5B4267F0
 P 9100 2950
-F 0 "#PWR26" H 9100 2700 50  0001 C CNN
+F 0 "#PWR020" H 9100 2700 50  0001 C CNN
 F 1 "GND" H 9100 2800 50  0000 C CNN
 F 2 "" H 9100 2950 50  0001 C CNN
@@
 CV
 $Comp
-L 2N3904 Q1
-U 1 1 5B42C9F8
-P 3750 1200
-F 0 "Q1" H 3950 1275 50  0000 L CNN
-F 1 "2N3904" H 3950 1200 50  0000 L CNN
-F 2 "TO_SOT_Packages_THT:TO-92_Molded_Narrow" H 3950 1125 50  0001 L CIN
-F 3 "" H 3750 1200 50  0001 L CNN
-	1    3750 1200
-	1    0    0    -1
-$EndComp
-$Comp
 L Audio-Jack-2_Switch J1
 U 1 1 5B42CA74
@@
 $EndComp
 $Comp
-L GND #PWR4
+L GND #PWR021
 U 1 1 5B42D1E5
 P 3500 1650
-F 0 "#PWR4" H 3500 1400 50  0001 C CNN
+F 0 "#PWR021" H 3500 1400 50  0001 C CNN
 F 1 "GND" H 3500 1500 50  0000 C CNN
 F 2 "" H 3500 1650 50  0001 C CNN
@@
 Text Label 7250 2950 2    60   ~ 0
 CLOCK
-$Comp
-L 2N3904 Q2
-U 1 1 5B42F247
-P 5700 1200
-F 0 "Q2" H 5900 1275 50  0000 L CNN
-F 1 "2N3904" H 5900 1200 50  0000 L CNN
-F 2 "TO_SOT_Packages_THT:TO-92_Molded_Narrow" H 5900 1125 50  0001 L CIN
-F 3 "" H 5700 1200 50  0001 L CNN
-	1    5700 1200
-	1    0    0    -1
-$EndComp
 $Comp
 L Audio-Jack-2_Switch J3
@@
 $EndComp
 $Comp
-L GND #PWR10
+L GND #PWR022
 U 1 1 5B42F267
 P 5450 1650
-F 0 "#PWR10" H 5450 1400 50  0001 C CNN
+F 0 "#PWR022" H 5450 1400 50  0001 C CNN
 F 1 "GND" H 5450 1500 50  0000 C CNN
 F 2 "" H 5450 1650 50  0001 C CNN
@@
 	3050 2750 3050 2950
 $Comp
-L VEE #PWR18
+L VEE #PWR023
 U 1 1 5B4591D4
 P 8150 1750
-F 0 "#PWR18" H 8150 1600 50  0001 C CNN
+F 0 "#PWR023" H 8150 1600 50  0001 C CNN
 F 1 "VEE" H 8150 1900 50  0000 C CNN
 F 2 "" H 8150 1750 50  0001 C CNN
@@
 $EndComp
 $Comp
-L VCC #PWR17
+L VCC #PWR024
 U 1 1 5B4592C7
 P 8150 1100
-F 0 "#PWR17" H 8150 950 50  0001 C CNN
+F 0 "#PWR024" H 8150 950 50  0001 C CNN
 F 1 "VCC" H 8150 1250 50  0000 C CNN
 F 2 "" H 8150 1100 50  0001 C CNN
@@
 $EndComp
 $Comp
-L VCC #PWR19
+L VCC #PWR025
 U 1 1 5B464DA9
 P 8150 2500
-F 0 "#PWR19" H 8150 2350 50  0001 C CNN
+F 0 "#PWR025" H 8150 2350 50  0001 C CNN
 F 1 "VCC" H 8150 2650 50  0000 C CNN
 F 2 "" H 8150 2500 50  0001 C CNN
@@
 $EndComp
 $Comp
-L VEE #PWR20
+L VEE #PWR026
 U 1 1 5B464E37
 P 8150 3150
-F 0 "#PWR20" H 8150 3000 50  0001 C CNN
+F 0 "#PWR026" H 8150 3000 50  0001 C CNN
 F 1 "VEE" H 8150 3300 50  0000 C CNN
 F 2 "" H 8150 3150 50  0001 C CNN
@@
 $EndComp
 $Comp
-L GND #PWR23
+L GND #PWR027
 U 1 1 5B467D2B
 P 8600 4750
-F 0 "#PWR23" H 8600 4500 50  0001 C CNN
+F 0 "#PWR027" H 8600 4500 50  0001 C CNN
 F 1 "GND" H 8600 4600 50  0000 C CNN
 F 2 "" H 8600 4750 50  0001 C CNN
@@
 $EndComp
 $Comp
-L GND #PWR22
+L GND #PWR028
 U 1 1 5B467D96
 P 8600 4450
-F 0 "#PWR22" H 8600 4200 50  0001 C CNN
+F 0 "#PWR028" H 8600 4200 50  0001 C CNN
 F 1 "GND" H 8600 4300 50  0000 C CNN
 F 2 "" H 8600 4450 50  0001 C CNN
@@
 $EndComp
 $Comp
-L GND #PWR21
+L GND #PWR029
 U 1 1 5B467E01
 P 8600 4150
-F 0 "#PWR21" H 8600 3900 50  0001 C CNN
+F 0 "#PWR029" H 8600 3900 50  0001 C CNN
 F 1 "GND" H 8600 4000 50  0000 C CNN
 F 2 "" H 8600 4150 50  0001 C CNN
@@
 $EndComp
 $Comp
-L GND #PWR13
+L GND #PWR030
 U 1 1 5B46803B
 P 6750 3750
-F 0 "#PWR13" H 6750 3500 50  0001 C CNN
+F 0 "#PWR030" H 6750 3500 50  0001 C CNN
 F 1 "GND" H 6750 3600 50  0000 C CNN
 F 2 "" H 6750 3750 50  0001 C CNN
@@
 	0    -1   -1   0
 $EndComp
+$Comp
+L MMBT3904 Q2
+U 1 1 5B5326AD
+P 5700 1200
+F 0 "Q2" H 5900 1275 50  0000 L CNN
+F 1 "MMBT3904" H 5900 1200 50  0000 L CNN
+F 2 "TO_SOT_Packages_SMD:SOT-23" H 5900 1125 50  0001 L CIN
+F 3 "" H 5700 1200 50  0001 L CNN
+	1    5700 1200
+	1    0    0    -1
+$EndComp
+$Comp
+L MMBT3904 Q1
+U 1 1 5B5328EC
+P 3750 1200
+F 0 "Q1" H 3950 1275 50  0000 L CNN
+F 1 "MMBT3904" H 3950 1200 50  0000 L CNN
+F 2 "TO_SOT_Packages_SMD:SOT-23" H 3950 1125 50  0001 L CIN
+F 3 "" H 3750 1200 50  0001 L CNN
+	1    3750 1200
+	1    0    0    -1
+$EndComp
 $EndSCHEMATC

Commit message: Bug Fixes and panel updates
Parts:
- removed Action1: Action Button, Buttons_Switches_THT:SW_MEC_5GTH9, symbol SW_Push_Open_Dual_x2
- removed Lane1: Lane Button, Buttons_Switches_THT:SW_MEC_5GTH9, symbol SW_Push_Open_Dual_x2
- removed Left1: Left Button, Buttons_Switches_THT:SW_MEC_5GTH9, symbol SW_Push_Open_Dual_x2
- removed Right1: Right Button, Buttons_Switches_THT:SW_MEC_5GTH9, symbol SW_Push_Open_Dual_x2
- added Action1: Action Button, Buttons_Switches_THT:SW_MEC_5GTH9, symbol MEC_Push_Switch
- added Lane1: Lane Button, Buttons_Switches_THT:SW_MEC_5GTH9, symbol MEC_Push_Switch
- added Left1: Left Button, Buttons_Switches_THT:SW_MEC_5GTH9, symbol MEC_Push_Switch
- added Right1: Right Button, Buttons_Switches_THT:SW_MEC_5GTH9, symbol MEC_Push_Switch
Connections:
- net ACTION: now also Action1.2
- net GND: now also Action1.3, Lane1.3, Left1.3, Right1.3
- net LANE: now also Lane1.2
- net LEFT: now also Left1.2
- net RIGHT: now also Right1.2
Changed lines of the file:
@@
-$EndComp
-$Comp
-L SW_Push_Open_Dual_x2 Right1
-U 1 1 5A99E833
-P 8300 4750
-F 0 "Right1" H 8300 4850 50  0000 C CNN
-F 1 "Right Button" H 8300 4675 50  0000 C CNN
-F 2 "Buttons_Switches_THT:SW_MEC_5GTH9" H 8300 4950 50  0001 C CNN
-F 3 "" H 8300 4950 50  0001 C CNN
-	1    8300 4750
-	-1   0    0    -1
-$EndComp
-$Comp
-L SW_Push_Open_Dual_x2 Left1
-U 1 1 5A99E8D7
-P 8300 5050
-F 0 "Left1" H 8300 5150 50  0000 C CNN
-F 1 "Left Button" H 8300 4975 50  0000 C CNN
-F 2 "Buttons_Switches_THT:SW_MEC_5GTH9" H 8300 5250 50  0001 C CNN
-F 3 "" H 8300 5250 50  0001 C CNN
-	1    8300 5050
-	-1   0    0    -1
 $EndComp
 $Comp
@@
 P 3700 2650
 F 0 "D1" H 3700 2750 50  0000 C CNN
-F 1 "1N5817" H 3700 2550 50  0000 C CNN
+F 1 "1N5817" H 3450 2700 50  0000 C CNN
 F 2 "Diodes_THT:D_DO-41_SOD81_P7.62mm_Horizontal" H 3700 2650 50  0001 C CNN
 F 3 "" H 3700 2650 50  0001 C CNN
@@
 $EndComp
 $Comp
-L SW_Push_Open_Dual_x2 Lane1
-U 1 1 5B422EFA
-P 8300 4450
-F 0 "Lane1" H 8300 4550 50  0000 C CNN
-F 1 "Lane Button" H 8300 4375 50  0000 C CNN
-F 2 "Buttons_Switches_THT:SW_MEC_5GTH9" H 8300 4650 50  0001 C CNN
-F 3 "" H 8300 4650 50  0001 C CNN
-	1    8300 4450
-	-1   0    0    -1
-$EndComp
-$Comp
 L GND #PWR015
 U 1 1 5B423678
@@
 	1    9150 5050
 	1    0    0    -1
-$EndComp
-$Comp
-L SW_Push_Open_Dual_x2 Action1
-U 1 1 5B423AB9
-P 8300 4150
-F 0 "Action1" H 8300 4250 50  0000 C CNN
-F 1 "Action Button" H 8300 4100 50  0000 C CNN
-F 2 "Buttons_Switches_THT:SW_MEC_5GTH9" H 8300 4350 50  0001 C CNN
-F 3 "" H 8300 4350 50  0001 C CNN
-	1    8300 4150
-	-1   0    0    -1
 $EndComp
 $Comp
@@
 P 3350 2850
 F 0 "J2" H 3400 3150 50  0000 C CNN
-F 1 "Eurorack_10_pin_power" H 3400 2550 50  0000 C CNN
+F 1 "Eurorack_10_pin_power" H 3450 2550 50  0000 C CNN
 F 2 "PlayDice:Multicomp_MC9A12-1034_2x05x2.54mm_Straight" H 3350 2850 50  0001 C CNN
 F 3 "" H 3350 2850 50  0001 C CNN
@@
 	1    0    0    -1
 $EndComp
+$Comp
+L MEC_Push_Switch Action1
+U 1 1 5B7990CD
+P 8300 4150
+F 0 "Action1" H 8300 4250 50  0000 C CNN
+F 1 "Action Button" H 8300 4075 50  0000 C CNN
+F 2 "Buttons_Switches_THT:SW_MEC_5GTH9" H 8300 4350 50  0001 C CNN
+F 3 "" H 8300 4350 50  0001 C CNN
+	1    8300 4150
+	1    0    0    -1
+$EndComp
+$Comp
+L MEC_Push_Switch Lane1
+U 1 1 5B79A837
+P 8300 4450
+F 0 "Lane1" H 8300 4550 50  0000 C CNN
+F 1 "Lane Button" H 8300 4375 50  0000 C CNN
+F 2 "Buttons_Switches_THT:SW_MEC_5GTH9" H 8300 4650 50  0001 C CNN
+F 3 "" H 8300 4650 50  0001 C CNN
+	1    8300 4450
+	1    0    0    -1
+$EndComp
+$Comp
+L MEC_Push_Switch Right1
+U 1 1 5B79A9AB
+P 8300 4750
+F 0 "Right1" H 8300 4850 50  0000 C CNN
+F 1 "Right Button" H 8300 4675 50  0000 C CNN
+F 2 "Buttons_Switches_THT:SW_MEC_5GTH9" H 8300 4950 50  0001 C CNN
+F 3 "" H 8300 4950 50  0001 C CNN
+	1    8300 4750
+	1    0    0    -1
+$EndComp
+$Comp
+L MEC_Push_Switch Left1
+U 1 1 5B79AB65
+P 8300 5050
+F 0 "Left1" H 8300 5150 50  0000 C CNN
+F 1 "Left Button" H 8300 4975 50  0000 C CNN
+F 2 "Buttons_Switches_THT:SW_MEC_5GTH9" H 8300 5250 50  0001 C CNN
+F 3 "" H 8300 5250 50  0001 C CNN
+	1    8300 5050
+	1    0    0    -1
+$EndComp

Commit message: Various code tidy-ups. Added configuration option for encoder direction. ADded new panel gerbers
Parts:
- Action1, Lane1, Left1, Right1: symbol MEC_Push_Switch -> PlayDice-rescue:MEC_Push_Switch
- C1, C2, C3, C4: symbol CP -> Device:CP
- D1, D2: symbol D -> Device:D
- Encoder1: symbol Rotary_Encoder_Switch -> PlayDice-rescue:Rotary_Encoder_Switch
- J1, J3, J5, J6: symbol Audio-Jack-2_Switch -> conn:Audio-Jack-2_Switch
- J2: symbol Eurorack_10_pin_power -> PlayDice-rescue:Eurorack_10_pin_power
- J4: symbol OLED -> PlayDice-rescue:OLED
- Q1, Q2: symbol MMBT3904 -> transistors:MMBT3904
- R1, R2, R3, R4, R5, R6, R7, R8: symbol R -> Device:R
- Teensy1: symbol Teensy3.2 -> teensy:Teensy3.2
- Tempo1: symbol POT -> PlayDice-rescue:POT
- U1: symbol LM1117-5.0 -> regul:LM1117-5.0
- U3: symbol TL072 -> linear:TL072
