File: Hardware/PlayDice.sch (KiCad schematic (older format))
At the start: 31 parts, among them J1 Clock In, J2 Eurorack_10_pin_power, J3 Action In, J4 OLED, J5 Gate Out, J6 CV Out, Q1 MMBT3904, Q2 MMBT3904, U1 LM1117-5.0, U3 TL072

Commit message: Revised Panel; started transferring Kicad files to v 5.99
Parts:
- Action1, Lane1, Left1, Right1: symbol MEC_Push_Switch -> PlayDice-rescue:MEC_Push_Switch
- C1, C2, C3, C4: symbol CP -> Device:CP
- D1, D2: symbol D -> Device:D
- Encoder1: symbol Rotary_Encoder_Switch -> PlayDice-rescue:Rotary_Encoder_Switch
- J1, J3, J5, J6: symbol Audio-Jack-2_Switch -> conn:Audio-Jack-2_Switch
- J2: symbol Eurorack_10_pin_power -> PlayDice-rescue:Eurorack_10_pin_power
- J4: symbol OLED -> PlayDice-rescue:OLED
- Q1, Q2: symbol MMBT3904 -> transistors:MMBT3904
- R1, R2, R3, R4, R5, R6, R7, R8: symbol R -> Device:R
- Teensy1: symbol Teensy3.2 -> teensy:Teensy3.2
- Tempo1: symbol POT -> PlayDice-rescue:POT
- U1: symbol LM1117-5.0 -> regul:LM1117-5.0
- U3: symbol TL072 -> linear:TL072
Connections:
- wire segments 91 -> 107
