File: Hardware/Panel.kicad_pcb (KiCad board)
At the start: 2 copper layers, 40.3 x 128.5 mm, 13 parts

Commit message: Updated to black and silver colour scheme; Transferred pcb and panel to Kicad 5.99
Other:
- board text added: "JLCJLCJLCJLC"
- board text added: "Play Dice Panel v2.0 Mountjoy Modular 2021"
Changed lines of the file:
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@@
   )
   (setup
+    (stackup
+      (layer "F.SilkS" (type "Top Silk Screen") (color "White"))
+      (layer "F.Paste" (type "Top Solder Paste"))
+      (layer "F.Mask" (type "Top Solder Mask") (color "Black") (thickness 0.01))
+      (layer "F.Cu" (type "copper") (thickness 0.035))
+      (layer "dielectric 1" (type "core") (thickness 1.51) (material "FR4") (epsilon_r 4.5) (loss_tangent 0.02))
+      (layer "B.Cu" (type "copper") (thickness 0.035))
+      (layer "B.Mask" (type "Bottom Solder Mask") (color "Black") (thickness 0.01))
+      (layer "B.Paste" (type "Bottom Solder Paste"))
+      (layer "B.SilkS" (type "Bottom Silk Screen") (color "White"))
+      (copper_finish "None")
+      (dielectric_constraints no)
+    )
     (pad_to_mask_clearance 0.2)
-    (aux_axis_origin 143.2 40)
-    (grid_origin 103 40)
     (pcbplotparams
-      (layerselection 0x00010f0_80000001)
+      (layerselection 0x00010f0_ffffffff)
       (disableapertmacros false)
       (usegerberextensions false)
@@
   (gr_circle (center 109.75 83.25) (end 113.830441 83.25) (layer "B.Mask") (width 1) (fill none))
   (gr_circle (center 111.3 130.7) (end 115.380441 130.7) (layer "B.Mask") (width 1) (fill none))
-  (gr_circle (center 84.4 123.4) (end 85.2 123.4) (layer "B.Mask") (width 0.2) (fill solid))
   (gr_rect (start 127.6 145.4) (end 118.4 154.6) (layer "B.Mask") (width 0.8) (fill solid))
   (gr_circle (center 135.75 83.25) (end 139.830441 83.25) (layer "B.Mask") (width 1) (fill none))
-  (gr_circle (center 75.9 114.8) (end 76.7 114.8) (layer "B.Mask") (width 0.2) (fill solid))
-  (gr_circle (center 75.9 123.4) (end 76.7 123.4) (layer "B.Mask") (width 0.2) (fill solid))
-  (gr_circle (center 80.2 119.1) (end 81 119.1) (layer "B.Mask") (width 0.2) (fill solid))
-  (gr_circle (center 84.4 114.8) (end 85.2 114.8) (layer "B.Mask") (width 0.2) (fill solid))
+  (gr_line (start 123.05 40) (end 123.05 168.5) (layer "Dwgs.User") (width 0.1))
   (gr_line (start 102.9 40) (end 143.2 40) (angle 90) (layer "Edge.Cuts") (width 0.15))
   (gr_line (start 143.2 40) (end 143.2 168.5) (angle 90) (layer "Edge.Cuts") (width 0.15))
@@
   (gr_line (start 110.4 56.9) (end 135.7 56.9) (angle 90) (layer "Edge.Cuts") (width 0.15))
   (gr_line (start 135.7 69.9) (end 110.4 69.9) (angle 90) (layer "Edge.Cuts") (width 0.15))
-  (gr_text "Lane\n" (at 122.9 75.469966) (layer "B.Mask")
+  (gr_text "Play Dice Panel v2.0\nMountjoy Modular 2021" (at 123.1 45.75) (layer "F.SilkS")
+    (effects (font (size 1 1) (thickness 0.15)))
+  )
+  (gr_text "JLCJLCJLCJLC" (at 123.05 163.8) (layer "F.SilkS")
+    (effects (font (size 1 1) (thickness 0.15)) (justify mirror))
+  )
+  (gr_text "Lane\n" (at 122.75 75.469966) (layer "B.Mask")
     (effects (font (size 1.5 1.5) (thickness 0.3)) (justify mirror))
   )
@@
   )
   (gr_text "Tempo" (at 132.5 111.9) (layer "B.Mask")
-    (effects (font (size 1.5 1.5) (thickness 0.3)) (justify mirror))
+    (effects (font (size 2 2) (thickness 0.3)) (justify mirror))
   )
   (gr_text "Clock In" (at 135.9 157.8) (layer "B.Mask")
@@
   )
   (gr_text "Edit" (at 113.5 111.9) (layer "B.Mask")
-    (effects (font (size 1.5 1.5) (thickness 0.3)) (justify mirror))
+    (effects (font (size 2 2) (thickness 0.3)) (justify mirror))
   )
   (gr_text "Gate Out" (at 123 157.8) (layer "B.Mask")
@@
     (effects (font (size 1.5 1.5) (thickness 0.3)) (justify mirror))
   )
-  (gr_text "Left" (at 135.7 75.5) (layer "B.Mask")
+  (gr_text "Left" (at 135.75 75.5) (layer "B.Mask")
     (effects (font (size 1.5 1.5) (thickness 0.3)) (justify mirror))
   )
-  (gr_text "Right" (at 109.6 75.5) (layer "B.Mask")
+  (gr_text "Right" (at 109.75 75.5) (layer "B.Mask")
     (effects (font (size 1.5 1.5) (thickness 0.3)) (justify mirror))
   )
@@
   (zone (net 0) (net_name "") (layer "F.Cu") (hatch edge 0.508)
     (connect_pads (clearance 0.508))
-    (min_thickness 0.254)
+    (min_thickness 0.254) (filled_areas_thickness no)
     (fill yes (thermal_gap 0.508) (thermal_bridge_width 0.508))
     (polygon
@@
   (zone (net 0) (net_name "") (layer "B.Cu") (hatch edge 0.508)
     (connect_pads (clearance 0.508))
-    (min_thickness 0.254)
+    (min_thickness 0.254) (filled_areas_thickness no)
     (fill yes (thermal_gap 0.508) (thermal_bridge_width 0.508))
     (polygon

Commit message: Panel pcb gerbers prepared for production
Other:
- rule pad_to_mask_clearance: 0.2 -> 0
Changed lines of the file:
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@@
       (layer "B.Paste" (type "Bottom Solder Paste"))
       (layer "B.SilkS" (type "Bottom Silk Screen") (color "White"))
-      (copper_finish "None")
+      (copper_finish "HAL lead-free")
       (dielectric_constraints no)
     )
-    (pad_to_mask_clearance 0.2)
+    (pad_to_mask_clearance 0)
     (pcbplotparams
       (layerselection 0x00010f0_ffffffff)
@@
       (usegerberextensions false)
       (usegerberattributes true)
-      (usegerberadvancedattributes true)
-      (creategerberjobfile true)
+      (usegerberadvancedattributes false)
+      (creategerberjobfile false)
       (svguseinch false)
       (svgprecision 6)
@@
       (plotinvisibletext false)
       (sketchpadsonfab false)
-      (subtractmaskfromsilk true)
+      (subtractmaskfromsilk false)
       (outputformat 1)
       (mirror false)
       (drillshape 0)
       (scaleselection 1)
-      (outputdirectory "Panel Gerbers/")
+      (outputdirectory "Gerbers/Panel/")
     )
   )
